Commit message: xacro

File: src/basic_description/urdf/basic_urdf.urdf.xacro (robot description, xacro)
@@ -1,4 +1,10 @@
 <?xml version="1.0"?>
-<robot name="basic_robot" xmlns:xacrp="http://www.ros.org/wiki/xacro">
+<robot name="basic_robot" xmlns:xacro="http://www.ros.org/wiki/xacro">
+  <xacro:property name="base_length" value="0.6" />
+  <xacro:property name="base_width" value="0.4" />
+  <xacro:property name="base_height" value="0.2" />
+  <xacro:property name="wheel_radius" value="0.1" />
+  <xacro:property name="wheel_length" value="0.05" />
+  <xacro:property name="caster_radius" value="0.05" />
   <material name="green">
     <color rgba="0 0.5 0 1" />
@@ -11,7 +17,7 @@
     <visual>
       <geometry>
-        <box size="0.6 0.4 0.2" />
+        <box size="${base_length} ${base_width} ${base_height}" />
       </geometry>
-      <origin xyz="0 0 0.1" rpy="0 0 0" />
+      <origin xyz="0 0 ${base_height/2}" rpy="0 0 0" />
       <material name="green" />
     </visual>
@@ -20,7 +26,7 @@
     <visual>
       <geometry>
-        <cylinder radius="0.1" length="0.2" />
+        <cylinder radius="${wheel_radius}" length="${base_height}" />
       </geometry>
-      <origin xyz="0 0 0.1" rpy="0 0 0" />
+      <origin xyz="0 0 ${base_height/2}" rpy="0 0 0" />
       <material name="grey" />
     </visual>
@@ -38,7 +44,7 @@
     <visual>
       <geometry>
-        <cylinder radius="0.1" length="0.05" />
+        <cylinder radius="${wheel_radius}" length="${wheel_length}" />
       </geometry>
-      <origin xyz="0 0 0" rpy="1.57 0 0" />
+      <origin xyz="0 0 0" rpy="${pi/2} 0 0" />
       <material name="grey" />
     </visual>
@@ -47,7 +53,7 @@
     <visual>
       <geometry>
-        <cylinder radius="0.1" length="0.05" />
+        <cylinder radius="${wheel_radius}" length="${wheel_length}" />
       </geometry>
-      <origin xyz="0 0 0" rpy="1.57 0 0" />
+      <origin xyz="0 0 0" rpy="${pi/2} 0 0" />
       <material name="grey" />
     </visual>
@@ -56,5 +62,5 @@
     <visual>
       <geometry>
-        <sphere radius="0.05" />
+        <sphere radius="${caster_radius}" />
       </geometry>
       <origin xyz="0 0 0.1" rpy="0 0 0" />
@@ -65,20 +71,20 @@
     <parent link="base_footprint" />
     <child link="base_link" />
-    <origin xyz="0 0 0.1" rpy="0 0 0"/>
+    <origin xyz="0 0 ${base_height/2}" rpy="0 0 0"/>
   </joint>
   <joint name="base_second_joint" type="fixed">
     <parent link="base_link" />
     <child link="second_link" />
-    <origin xyz="0 0 0.2" rpy="0 0 0" />
+    <origin xyz="0 0 ${base_height}" rpy="0 0 0" />
   </joint>
   <joint name="second_third_joint" type="fixed">
     <parent link="second_link" />
     <child link="third_link" />
-    <origin xyz="0 0 0.2" rpy="0 0 0" />
+    <origin xyz="0 0 ${base_height}" rpy="0 0 0" />
   </joint>
   <joint name="base_right_wheel_joint" type="continuous">
     <parent link="base_link" />
     <child link="right_wheel_link" />
-    <origin xyz="-0.15 -0.225 0" rpy="0 0 0" />
+    <origin xyz="${-base_length/4.0} -0.225 0" rpy="0 0 0" />
     <axis xyz="0 1 0" />
   </joint>
@@ -86,5 +92,5 @@
     <parent link="base_link" />
     <child link="left_wheel_link" />
-    <origin xyz="-0.15 0.225 0" rpy="0 0 0" />
+    <origin xyz="${-base_length/4.0} 0.225 0" rpy="0 0 0" />
     <axis xyz="0 1 0" />
   </joint>
@@ -92,5 +98,5 @@
     <parent link="base_link" />
     <child link="caster_wheel_link" />
-    <origin xyz="0.2 0 -0.05" rpy="0 0 0" />
+    <origin xyz="${base_length/3.0} 0 -0.05" rpy="0 0 0" />
   </joint>
 </robot>

Commit message: gazebo

File: src/basic_description/urdf/basic_urdf.urdf.xacro (robot description, xacro)
@@ -13,4 +13,31 @@
     <color rgba="0.5 0.5 0.5 1" />
   </material>
+  <xacro:macro name="box_inertia" params="m x y z xyz rpy">
+    <inertial>
+      <origin xyz="${xyz}" rpy="${rpy}"/>
+      <mass value="${m}"/>
+      <inertia ixx="${(m/12) * (y*y + z*z)}" ixy="0.0" ixz="0.0"
+               iyy="${(m/12) * (x*x + z*z)}" iyz="0.0"
+               izz="${(m/12) * (x*x + y*y)}"/>
+    </inertial>
+  </xacro:macro>
+  <xacro:macro name="cylinder_inertia" params="m r h xyz rpy">
+    <inertial>
+      <origin xyz="${xyz}" rpy="${rpy}"/>
+      <mass value="${m}"/>
+      <inertia ixx="${(m/12) * (3*r*r + h*h)}" ixy="0.0" ixz="0.0"
+               iyy="${(m/12) * (3*r*r + h*h)}" iyz="0.0"
+               izz="${(m/2) * (r*r)}"/>
+    </inertial>
+  </xacro:macro>
+  <xacro:macro name="sphere_inertia" params="m r xyz rpy">
+    <inertial>
+      <origin xyz="${xyz}" rpy="${rpy}"/>
+      <mass value="${m}"/>
+      <inertia ixx="${(2/5) * m * (r*r)}" ixy="0.0" ixz="0.0"
+               iyy="${(2/5) * m * (r*r)}" iyz="0.0"
+               izz="${(2/5) * m * (r*r)}"/>
+    </inertial>
+  </xacro:macro>
   <link name="base_footprint" />
   <link name="base_link">
@@ -22,4 +49,11 @@
       <material name="green" />
     </visual>
+    <collision>
+      <geometry>
+        <box size="${base_length} ${base_width} ${base_height}" />
+      </geometry>
+      <origin xyz="0 0 ${base_height/2}" rpy="0 0 0" />
+    </collision>
+    <xacro:box_inertia m="5.0" x="${base_length}" y="${base_width}" z="${base_height}" xyz="0 0 ${base_height/2}" rpy="0 0 0" />
   </link>
   <link name="second_link">
@@ -31,4 +65,11 @@
       <material name="grey" />
     </visual>
+    <collision>
+      <geometry>
+        <sphere radius="${wheel_radius}" />
+      </geometry>
+      <origin xyz="0 0 ${base_height/2}" rpy="0 0 0" />
+    </collision>
+    <xacro:cylinder_inertia m="1.0" r="${wheel_radius}" h="${base_height}" xyz="0 0 ${base_height/2}" rpy="0 0 0" />
   </link>
   <link name="third_link">
@@ -40,4 +81,11 @@
       <material name="green" />
     </visual>
+    <collision>
+      <geometry>
+        <box size="0.1 0.1 0.1" />
+      </geometry>
+      <origin xyz="0 0 0.05" rpy="0 0 0" />
+    </collision>
+    <xacro:box_inertia m="0.5" x="0.1" y="0.1" z="0.1" xyz="0 0 0.05" rpy="0 0 0" />
   </link>
   <link name="right_wheel_link">
@@ -49,4 +97,11 @@
       <material name="grey" />
     </visual>
+    <collision>
+      <geometry>
+        <sphere radius="${wheel_radius}" />
+      </geometry>
+      <origin xyz="0 0 0" rpy="${pi/2} 0 0" />
+    </collision>
+    <xacro:cylinder_inertia m="1.0" r="${wheel_radius}" h="${wheel_length}" xyz="0 0 0" rpy="${pi/2} 0 0" />
   </link>
   <link name="left_wheel_link">
@@ -58,4 +113,11 @@
       <material name="grey" />
     </visual>
+    <collision>
+      <geometry>
+        <sphere radius="${wheel_radius}" />
+      </geometry>
+      <origin xyz="0 0 0" rpy="${pi/2} 0 0" />
+    </collision>
+    <xacro:cylinder_inertia m="1.0" r="${wheel_radius}" h="${wheel_length}" xyz="0 0 0" rpy="${pi/2} 0 0" />
   </link>
   <link name="caster_wheel_link">
@@ -64,7 +126,14 @@
         <sphere radius="${caster_radius}" />
       </geometry>
-      <origin xyz="0 0 0.1" rpy="0 0 0" />
+      <origin xyz="0 0 0" rpy="0 0 0" />
       <material name="grey" />
     </visual>
+    <collision>
+      <geometry>
+        <sphere radius="${caster_radius}" />
+      </geometry>
+      <origin xyz="0 0 0" rpy="0 0 0" />
+    </collision>
+    <xacro:sphere_inertia m="0.5" r="${caster_radius}" xyz="0 0 0" rpy="0 0 0" />
   </link>
   <joint name="base_joint" type="fixed">

Commit message: camea sensors

File: src/basic_description/urdf/basic_urdf.urdf.xacro (robot description, xacro)
@@ -137,4 +137,5 @@
     <xacro:sphere_inertia m="0.5" r="${caster_radius}" xyz="0 0 0" rpy="0 0 0" />
   </link>
+  <link name="camera_link_optical" />
   <joint name="base_joint" type="fixed">
     <parent link="base_footprint" />
@@ -168,4 +169,9 @@
     <child link="caster_wheel_link" />
     <origin xyz="${base_length/3.0} 0 -0.05" rpy="0 0 0" />
+  </joint>
+  <joint name="camera_optical_joint" type="fixed">
+    <origin xyz="0 0 0" rpy="${-pi/2} 0 ${-pi/2}" />
+    <parent link="third_link" />
+    <child link="camera_link_optical" />
   </joint>
   <gazebo reference="caster_wheel_link">
@@ -189,3 +195,30 @@
     </plugin>
   </gazebo>
+  <gazebo reference="third_link">
+    <sensor name="camera" type="camera">
+      <camera>
+        <horizontal_fov>1.3962634</horizontal_fov>
+        <image>
+          <width>640</width>
+          <heigth>480</heigth>
+          <format>R8G8B8</format>
+        </image>
+        <clip>
+          <near>0.1</near>
+          <far>15</far>
+        </clip>
+        <noise>
+          <type>gaussian</type>
+          <mean>0.0</mean>
+          <stddev>0.007</stddev>
+        </noise>
+        <optical_frame_id>camera_link_optical</optical_frame_id>
+        <camera_info_topic>camera/camera_info</camera_info_topic>
+      </camera>
+      <always_on>1</always_on>
+      <update_rate>20</update_rate>
+      <visualize>true</visualize>
+      <topic>camera/image_raw</topic>
+    </sensor>
+  </gazebo>
 </robot>
